File: AirSensor_LoRA.sch (EAGLE design)
At the start: 6 parts, among them U2 RFM95W-915S2

Commit message: added JTAG schematic and PCB  + all pictures
Parts:
- added C1: 1uF, SparkFun-Capacitors:1.0UF-0805-25V-10%
- added C2: 10uF, SparkFun-Capacitors:1.0UF-0805-25V-10%
Connections:
- net GND: now also C1.2, C2.2
- net N$17: now also C1.1, C2.1
Changed lines of the file:
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@@
 <part name="C10" library="SparkFun-Capacitors" library_urn="urn:adsk.eagle:library:510" deviceset="1.0UF" device="-0805-25V-10%" package3d_urn="urn:adsk.eagle:package:37429/1" value="0.1uF"/>
 <part name="GND1" library="SparkFun-PowerSymbols" library_urn="urn:adsk.eagle:library:530" deviceset="GND" device=""/>
+<part name="GND2" library="SparkFun-Aesthetics" deviceset="GND" device=""/>
+<part name="C1" library="SparkFun-Capacitors" library_urn="urn:adsk.eagle:library:510" deviceset="1.0UF" device="-0805-25V-10%" package3d_urn="urn:adsk.eagle:package:37429/1" value="1uF"/>
+<part name="GND3" library="SparkFun-Aesthetics" deviceset="GND" device=""/>
+<part name="C2" library="SparkFun-Capacitors" library_urn="urn:adsk.eagle:library:510" deviceset="1.0UF" device="-0805-25V-10%" package3d_urn="urn:adsk.eagle:package:37429/1" value="10uF"/>
 </parts>
 <sheets>
@@
 <attribute name="VALUE" x="129.54" y="48.006" size="1.778" layer="96" align="top-center"/>
 </instance>
+<instance part="GND2" gate="1" x="144.78" y="76.2" smashed="yes">
+<attribute name="VALUE" x="142.24" y="73.66" size="1.778" layer="96"/>
+</instance>
+<instance part="C1" gate="G$1" x="144.78" y="83.82" smashed="yes">
+<attribute name="NAME" x="146.304" y="86.741" size="1.778" layer="95" font="vector"/>
+<attribute name="VALUE" x="146.304" y="81.661" size="1.778" layer="96" font="vector"/>
+</instance>
+<instance part="GND3" gate="1" x="152.4" y="76.2" smashed="yes">
+<attribute name="VALUE" x="149.86" y="73.66" size="1.778" layer="96"/>
+</instance>
+<instance part="C2" gate="G$1" x="152.4" y="83.82" smashed="yes">
+<attribute name="NAME" x="153.924" y="86.741" size="1.778" layer="95" font="vector"/>
+<attribute name="VALUE" x="153.924" y="81.661" size="1.778" layer="96" font="vector"/>
+</instance>
 </instances>
 <busses>
@@
 <junction x="129.54" y="53.34"/>
 </segment>
+<segment>
+<pinref part="GND2" gate="1" pin="GND"/>
+<wire x1="144.78" y1="78.74" x2="144.78" y2="81.28" width="0.1524" layer="91"/>
+<pinref part="C1" gate="G$1" pin="2"/>
+</segment>
+<segment>
+<pinref part="GND3" gate="1" pin="GND"/>
+<wire x1="152.4" y1="78.74" x2="152.4" y2="81.28" width="0.1524" layer="91"/>
+<pinref part="C2" gate="G$1" pin="2"/>
+</segment>
 </net>
 <net name="3.3V" class="0">
@@
 <wire x1="137.16" y1="91.44" x2="137.16" y2="88.9" width="0.1524" layer="91"/>
 <pinref part="C10" gate="G$1" pin="1"/>
+<wire x1="144.78" y1="91.44" x2="144.78" y2="88.9" width="0.1524" layer="91"/>
+<pinref part="C1" gate="G$1" pin="1"/>
+<wire x1="137.16" y1="91.44" x2="144.78" y2="91.44" width="0.1524" layer="91"/>
+<junction x="137.16" y="91.44"/>
+<wire x1="152.4" y1="91.44" x2="152.4" y2="88.9" width="0.1524" layer="91"/>
+<pinref part="C2" gate="G$1" pin="1"/>
+<wire x1="144.78" y1="91.44" x2="152.4" y2="91.44" width="0.1524" layer="91"/>
+<junction x="144.78" y="91.44"/>
 </segment>
 </net>

Commit message: nieuw schema lora bordje
Parts:
- removed C10: 0.1uF, SparkFun-Capacitors:1.0UF-0805-25V-10%
- removed RFM95W_1: LoRa_1, con-lstb:MA05-1
- removed RFM95W_2: LoRa_2, con-lstb:MA05-1
- removed S1: (no value), switch-omron:10-XX
- removed U2: RFM95W-915S2, RFM95W-915S2:RFM95W-915S2
- removed X1: (no value), adafruit:SMACONNECTOR_EDGE
- added C3: 10µ, Resistor_Capacitor:CC0805KRX7R9BB104
- added J1, J2: (no value), SparkFun-Connectors:CONN_05
- added LED1: (no value), adafruit:LEDCHIPLED_0805
- added MODULE1: RN2483-I/RM095, RN2483-I_RM095 (3):RN2483-I/RM095
- added R1: 10k, Resistor_Capacitor:CRCW08050000Z0EA
- added R2: 220, Resistor_Capacitor:CRCW08050000Z0EA
- C1: value 1uF -> 0.1µ; device SparkFun-Capacitors:1.0UF-0805-25V-10% -> Resistor_Capacitor:CC0805KRX7R9BB104
- C2: value 10uF -> 1µ; device SparkFun-Capacitors:1.0UF-0805-25V-10% -> Resistor_Capacitor:CC0805KRX7R9BB104
Connections:
- removed net 3.3V: S1.P, S1.P1
- removed net GND: C1.2, C10.2, C2.2, RFM95W_2.5, U2.GND, X1.GND1, X1.GND2, X1.GND3, X1.GND4
- removed net N$13: RFM95W_1.2, S1.S, S1.S1, U2.RESET
- removed net N$17: C1.1, C10.1, C2.1, RFM95W_2.1, U2.3.3V
- removed net N$18: RFM95W_2.2, U2.MOSI
- removed net N$21: RFM95W_2.3, U2.MISO
- removed net N$22: RFM95W_2.4, U2.NSS
- removed net N$23: RFM95W_1.5, U2.SCK
- removed net N$24: RFM95W_1.4, U2.DIO0
- removed net N$25: RFM95W_1.3, U2.DIO1
- removed net N$26: U2.ANT, X1.ANT
- new net N$1: J2.3, MODULE1.UART_RX
- new net N$2: J2.2, MODULE1.UART_TX
- new net N$3: J1.5, MODULE1.!RESET, R1.2
- new net N$4: C1.1, C2.1, C3.1, J1.3, MODULE1.VDD1, R1.1
- new net N$5: C1.2, C2.2, C3.2, J1.1, LED1.C, MODULE1.GND
- new net N$6: MODULE1.VDD2, R2.2
- new net N$8: LED1.A, R2.1
Other:
- moved on the sheet: C1, C2
