File: Moederbord/AirSensor.brd (EAGLE design)
At the start: 108.6 x 80 mm, 33 parts, among them J1 battery Output 7.4V, J3 2013499-1, Q1 2N7000, U1 ATSAMD21G18A-AU, U2 MIC5219 3.3V, Y1 32.768kHz

Commit message: added solar charger, PCB image, ...
Parts:
- removed J3: 2013499-1, 2013499-1:TE_2013499-1
- added J2: 10118194-0001LF, 10118194-0001LF:AMPHENOL_10118194-0001LF
- moved R4 16.9 mm to (69.7, 46.9), turned to 0 degrees
- moved Q1 12.9 mm to (68.8, 42.3), turned to 270 degrees
Connections:
- removed net VBUS: J3.1
- net B_FET: now also U1.15; no longer U1.24
- net D+: now also J2.3; no longer J3.3
- net D-: now also J2.2; no longer J3.2
- net GND: now also J2.5, J2.S1, J2.S2, J2.S3, J2.S4, J2.S5, J2.S6; no longer J3.10, J3.11, J3.5, J3.6, J3.7, J3.8, J3.9
- net RXD: now also U1.37; no longer U1.10
- net SCL: now also U1.14; no longer U1.32
- net SDA: now also U1.13; no longer U1.31
- net TXD: now also U1.38; no longer U1.9
Routing:
- net RXD: track 44.0 -> 56.6 mm
- net SDA: track 38.6 -> 45.0 mm
- net SCL: track 34.7 -> 39.5 mm
- net B_FET: track 12.7 -> 8.24 mm
- net GND: track 38.0 -> 33.9 mm
- net TXD: track 36.2 -> 38.5 mm
- net GND_FET: track 63.9 -> 63.1 mm
