File: Moederbord/AirSensor.sch (EAGLE design)
At the start: 33 parts, among them J1 battery Output 7.4V, J3 2013499-1, Q1 2N7000, U1 ATSAMD21G18A-AU, U2 MIC5219 3.3V, Y1 32.768kHz

Commit message: added solar charger, PCB image, ...
Parts:
- removed J3: 2013499-1, 2013499-1:2013499-1
- added J2: 10118194-0001LF, 10118194-0001LF:10118194-0001LF
Connections:
- net B_FET: now also U1.PA10; no longer U1.PA15
- net D+: now also J2.3; no longer J3.D+
- net D-: now also J2.2; no longer J3.D-
- net GND: now also J2.5, J2.SHIELD; no longer J3.GND, J3.SLD
- net RXD: now also U1.PB22; no longer U1.PA05
- net SCL: now also U1.PA09; no longer U1.PA23
- net SDA: now also U1.PA08; no longer U1.PA22
- net TXD: now also U1.PB23; no longer U1.PA04
Changed lines of the file:
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@@
 <part name="S1" library="EG1213" deviceset="EG1213" device=""/>
 <part name="GND8" library="SparkFun-Aesthetics" deviceset="GND" device=""/>
-<part name="J3" library="2013499-1" deviceset="2013499-1" device=""/>
 <part name="GND15" library="SparkFun-Aesthetics" deviceset="GND" device=""/>
+<part name="J2" library="10118194-0001LF" deviceset="10118194-0001LF" device=""/>
 </parts>
 <sheets>
@@
 <attribute name="VALUE" x="-10.16" y="45.72" size="1.778" layer="96"/>
 </instance>
-<instance part="J3" gate="G$1" x="114.3" y="99.06" smashed="yes" rot="R270">
-<attribute name="NAME" x="121.931790625" y="106.691790625" size="1.78075" layer="95" rot="R270"/>
-<attribute name="VALUE" x="104.1355" y="106.683390625" size="1.778790625" layer="96" rot="R270"/>
-</instance>
 <instance part="GND15" gate="1" x="109.22" y="132.08" smashed="yes" rot="R180">
 <attribute name="VALUE" x="111.76" y="134.62" size="1.778" layer="96" rot="R180"/>
+</instance>
+<instance part="J2" gate="G$1" x="111.76" y="93.98" smashed="yes" rot="R270">
+<attribute name="NAME" x="122.4349" y="101.355040625" size="1.271559375" layer="95" rot="R270"/>
+<attribute name="VALUE" x="99.0561" y="101.603940625" size="1.270659375" layer="96" rot="R270"/>
 </instance>
 </instances>
@@
 <segment>
 <pinref part="GND15" gate="1" pin="GND"/>
-<wire x1="109.22" y1="129.54" x2="109.22" y2="111.76" width="0.1524" layer="91"/>
-<pinref part="J3" gate="G$1" pin="GND"/>
-<pinref part="J3" gate="G$1" pin="SLD"/>
-<wire x1="109.22" y1="111.76" x2="109.22" y2="109.22" width="0.1524" layer="91"/>
-<wire x1="109.22" y1="88.9" x2="109.22" y2="83.82" width="0.1524" layer="91"/>
-<wire x1="109.22" y1="83.82" x2="101.6" y2="83.82" width="0.1524" layer="91"/>
-<wire x1="101.6" y1="83.82" x2="101.6" y2="111.76" width="0.1524" layer="91"/>
-<wire x1="101.6" y1="111.76" x2="109.22" y2="111.76" width="0.1524" layer="91"/>
-<junction x="109.22" y="111.76"/>
+<wire x1="109.22" y1="129.54" x2="109.22" y2="114.3" width="0.1524" layer="91"/>
+<pinref part="J2" gate="G$1" pin="5"/>
+<pinref part="J2" gate="G$1" pin="SHIELD"/>
+<wire x1="109.22" y1="114.3" x2="109.22" y2="106.68" width="0.1524" layer="91"/>
+<wire x1="104.14" y1="106.68" x2="104.14" y2="114.3" width="0.1524" layer="91"/>
+<wire x1="104.14" y1="114.3" x2="109.22" y2="114.3" width="0.1524" layer="91"/>
+<junction x="109.22" y="114.3"/>
 </segment>
 </net>
@@
 </segment>
 <segment>
-<pinref part="J3" gate="G$1" pin="D+"/>
-<wire x1="114.3" y1="109.22" x2="114.3" y2="116.84" width="0.1524" layer="91"/>
+<wire x1="114.3" y1="106.68" x2="114.3" y2="116.84" width="0.1524" layer="91"/>
 <label x="114.3" y="114.3" size="1.778" layer="95" rot="R90" align="bottom-right"/>
+<pinref part="J2" gate="G$1" pin="3"/>
 </segment>
 </net>
@@
 </segment>
 <segment>
-<pinref part="J3" gate="G$1" pin="D-"/>
-<wire x1="116.84" y1="109.22" x2="116.84" y2="116.84" width="0.1524" layer="91"/>
+<wire x1="116.84" y1="106.68" x2="116.84" y2="116.84" width="0.1524" layer="91"/>
 <label x="116.84" y="114.3" size="1.778" layer="95" rot="R90" align="bottom-right"/>
+<pinref part="J2" gate="G$1" pin="2"/>
 </segment>
 </net>
@@
 </segment>
 <segment>
-<pinref part="U1" gate="G$1" pin="PA15"/>
-<wire x1="35.56" y1="86.36" x2="22.86" y2="86.36" width="0.1524" layer="91"/>
-<label x="25.4" y="86.36" size="1.778" layer="95"/>
+<pinref part="U1" gate="G$1" pin="PA10"/>
+<wire x1="35.56" y1="99.06" x2="22.86" y2="99.06" width="0.1524" layer="91"/>
+<label x="25.4" y="99.06" size="1.778" layer="95"/>
 </segment>
 </net>
@@
 </segment>
 <segment>
-<pinref part="U1" gate="G$1" pin="PA05"/>
-<wire x1="35.56" y1="111.76" x2="25.4" y2="111.76" width="0.1524" layer="91"/>
-<label x="27.94" y="111.76" size="1.778" layer="95"/>
+<pinref part="U1" gate="G$1" pin="PB22"/>
+<wire x1="71.12" y1="93.98" x2="81.28" y2="93.98" width="0.1524" layer="91"/>
+<label x="78.74" y="93.98" size="1.778" layer="95" align="bottom-right"/>
 </segment>
 </net>
@@
 </segment>
 <segment>
-<pinref part="U1" gate="G$1" pin="PA04"/>
-<wire x1="35.56" y1="114.3" x2="25.4" y2="114.3" width="0.1524" layer="91"/>
-<label x="27.94" y="114.3" size="1.778" layer="95"/>
+<pinref part="U1" gate="G$1" pin="PB23"/>
+<wire x1="71.12" y1="91.44" x2="81.28" y2="91.44" width="0.1524" layer="91"/>
+<label x="78.74" y="91.44" size="1.778" layer="95" align="bottom-right"/>
 </segment>
 </net>
 <net name="SCL" class="0">
-<segment>
-<pinref part="U1" gate="G$1" pin="PA23"/>
-<wire x1="35.56" y1="66.04" x2="25.4" y2="66.04" width="0.1524" layer="91"/>
-<label x="27.94" y="66.04" size="1.778" layer="95"/>
-</segment>
 <segment>
 <pinref part="HIH8XXX" gate="G$1" pin="3"/>
@@
 <junction x="165.1" y="124.46"/>
 </segment>
+<segment>
+<pinref part="U1" gate="G$1" pin="PA09"/>
+<wire x1="35.56" y1="101.6" x2="25.4" y2="101.6" width="0.1524" layer="91"/>
+<label x="27.94" y="101.6" size="1.778" layer="95"/>
+</segment>
 </net>
 <net name="SDA" class="0">
@@
 </segment>
 <segment>
-<pinref part="U1" gate="G$1" pin="PA22"/>
-<wire x1="35.56" y1="68.58" x2="25.4" y2="68.58" width="0.1524" layer="91"/>
-<label x="27.94" y="68.58" size="1.778" layer="95"/>
-</segment>
-</net>
+<pinref part="U1" gate="G$1" pin="PA08"/>
+<wire x1="35.56" y1="104.14" x2="25.4" y2="104.14" width="0.1524" layer="91"/>
+<label x="27.94" y="104.14" size="1.778" layer="95"/>
+</segment>
+</net>
