File: LoRa/AirSensor_LoRA.brd (EAGLE design)
At the start: 37.8 x 45.1 mm, 11 parts

Commit message: rx/tx fout opgelost in PCB
Parts:
- turned RFM95W_2 to 270 degrees
Routing:
- net TXD: track 14.0 -> 21.9 mm
- net RXD: track 17.3 -> 13.1 mm
Changed lines of the file:
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@@
 </layers>
 <board>
-<fusionsync huburn="a.YnVzaW5lc3M6c2t5bmV0MTMz" projecturn="a.YnVzaW5lc3M6c2t5bmV0MTMzI0QyMDE5MTAzMTIzMzQxNDY3Ng" f3durn="urn:adsk.wipprod:dm.lineage:gBG1N-XqQO-DzMLJpc-8hg" pcbguid="" lastpulledtime="" lastsyncedchangeguid="" latestrevisionid="ac4a1052-f352-472b-a3a7-5576a45fbe37" lastsyncedrevisionid="ac4a1052-f352-472b-a3a7-5576a45fbe37" lastboardhashguid="241796fe-0e12-6c2b-dce0-969d89b7f3a3" lastpushedtime="2020-12-11T13:20:17Z" linktopcb3d="true"/>
+<fusionsync huburn="a.YnVzaW5lc3M6c2t5bmV0MTMz" projecturn="a.YnVzaW5lc3M6c2t5bmV0MTMzI0QyMDE5MTAzMTIzMzQxNDY3Ng" f3durn="urn:adsk.wipprod:dm.lineage:gBG1N-XqQO-DzMLJpc-8hg" pcbguid="" lastpulledtime="" lastsyncedchangeguid="" latestrevisionid="ac4a1052-f352-472b-a3a7-5576a45fbe37" lastsyncedrevisionid="ac4a1052-f352-472b-a3a7-5576a45fbe37" lastboardhashguid="241796fe-0e12-6c2b-dce0-969d89b7f3a3" lastpushedtime="2020-12-11T13:20:17Z" linktopcb3d="false"/>
 <plain>
 <wire x1="0" y1="52.2986" x2="37.77" y2="52.324" width="0" layer="20"/>
@@
 <attribute name="POPULARITY" value="29" x="-8.89" y="52.07" size="1.778" layer="27" rot="R270" display="off"/>
 </element>
-<element name="RFM95W_2" library="con-lstb" library_urn="urn:adsk.eagle:library:162" package="MA05-1" package3d_urn="urn:adsk.eagle:package:8332/1" value="LoRa_2" x="5.08" y="72.39" smashed="yes" rot="R90">
-<attribute name="MF" value="" x="46.99" y="106.68" size="1.778" layer="27" rot="R90" display="off"/>
-<attribute name="MPN" value="" x="46.99" y="106.68" size="1.778" layer="27" rot="R90" display="off"/>
-<attribute name="OC_FARNELL" value="unknown" x="46.99" y="106.68" size="1.778" layer="27" rot="R90" display="off"/>
-<attribute name="OC_NEWARK" value="unknown" x="46.99" y="106.68" size="1.778" layer="27" rot="R90" display="off"/>
-<attribute name="POPULARITY" value="29" x="46.99" y="106.68" size="1.778" layer="27" rot="R90" display="off"/>
+<element name="RFM95W_2" library="con-lstb" library_urn="urn:adsk.eagle:library:162" package="MA05-1" package3d_urn="urn:adsk.eagle:package:8332/1" value="LoRa_2" x="5.08" y="72.39" smashed="yes" rot="R270">
+<attribute name="MF" value="" x="-36.83" y="38.1" size="1.778" layer="27" rot="R270" display="off"/>
+<attribute name="MPN" value="" x="-36.83" y="38.1" size="1.778" layer="27" rot="R270" display="off"/>
+<attribute name="OC_FARNELL" value="unknown" x="-36.83" y="38.1" size="1.778" layer="27" rot="R270" display="off"/>
+<attribute name="OC_NEWARK" value="unknown" x="-36.83" y="38.1" size="1.778" layer="27" rot="R270" display="off"/>
+<attribute name="POPULARITY" value="29" x="-36.83" y="38.1" size="1.778" layer="27" rot="R270" display="off"/>
 </element>
 <element name="S1" library="switch-omron" library_urn="urn:adsk.eagle:library:377" package="B3F-10XX" package3d_urn="urn:adsk.eagle:package:27496/1" value="" x="14.4272" y="56.5912" smashed="yes">
@@
 <wire x1="10.16" y1="84.709" x2="10.1346" y2="84.6836" width="0.4064" layer="1"/>
 <wire x1="10.1346" y1="84.6836" x2="9.63170625" y2="84.6836" width="0.4064" layer="1"/>
-<wire x1="5.08" y1="70.04746875" x2="5.08" y2="69.85" width="0.4064" layer="1"/>
-<wire x1="9.63170625" y1="84.6836" x2="7.7978" y2="82.84969375" width="0.4064" layer="1"/>
-<wire x1="7.7978" y1="82.84969375" x2="7.7978" y2="72.76526875" width="0.4064" layer="1"/>
-<wire x1="7.7978" y1="72.76526875" x2="5.08" y2="70.04746875" width="0.4064" layer="1"/>
+<wire x1="7.366" y1="75.692" x2="6.604" y2="74.93" width="0.4064" layer="1"/>
+<wire x1="6.604" y1="74.93" x2="5.08" y2="74.93" width="0.4064" layer="1"/>
+<wire x1="9.63170625" y1="84.6836" x2="7.366" y2="82.41789375" width="0.4064" layer="1"/>
+<wire x1="7.366" y1="82.41789375" x2="7.366" y2="75.692" width="0.4064" layer="1"/>
 </signal>
 <signal name="TXD">
 <contactref element="MODULE1" pad="6"/>
 <contactref element="RFM95W_2" pad="4"/>
-<wire x1="5.08" y1="74.93" x2="6.985" y2="76.835" width="0.4064" layer="1"/>
-<wire x1="6.985" y1="76.835" x2="6.985" y2="84.201" width="0.4064" layer="1"/>
-<wire x1="6.985" y1="84.201" x2="8.763" y2="85.979" width="0.4064" layer="1"/>
-<wire x1="8.763" y1="85.979" x2="10.16" y2="85.979" width="0.4064" layer="1"/>
+<wire x1="5.08" y1="69.85" x2="3.683" y2="69.85" width="0.4064" layer="1"/>
+<wire x1="3.683" y1="69.85" x2="2.921" y2="70.612" width="0.4064" layer="1"/>
+<wire x1="2.921" y1="70.612" x2="2.921" y2="80.518" width="0.4064" layer="1"/>
+<wire x1="2.921" y1="80.518" x2="3.175" y2="80.772" width="0.4064" layer="1"/>
+<wire x1="8.382" y1="85.979" x2="3.175" y2="80.772" width="0.4064" layer="1"/>
+<wire x1="10.16" y1="85.979" x2="8.382" y2="85.979" width="0.4064" layer="1"/>
 </signal>
 <signal name="ANT">
